Commit message: Sim completed for KPIs

File: install/qcar_description/share/qcar_description/urdf/qcar.urdf.xacro (robot description, xacro)
@@ -1 +1,36 @@
-/home/g16/Documents/qcarSim/src/qcar_description/urdf/qcar.urdf.xacro
+<?xml version='1.0'?>
+<robot name="qcar" xmlns:xacro="http://www.ros.org/wiki/xacro">
+  <xacro:arg name="components_config" default="$(find qcar_description)/config/qcar/basic.yaml" />
+  <xacro:arg name="configuration" default="basic" />
+  <xacro:arg name="controller_config" default="" />
+  <xacro:arg name="namespace" default="" />
+  <xacro:arg name="use_sim" default="False" />
+  <xacro:include filename="$(find qcar_description)/urdf/qcar_body.urdf.xacro" ns="body" />
+  <xacro:include filename="$(find qcar_description)/urdf/qcar_wheels.urdf.xacro" ns="wheel" />
+  <xacro:include filename="$(find qcar_description)/urdf/qcar_gz.urdf.xacro" ns="gz" />
+  <!-- PROPERTIES -->
+  <xacro:property name="wheel_radius" value="0.033" />
+  <!-- BODY -->
+  <xacro:body.body wheel_radius="${wheel_radius}" namespace="$(arg namespace)" />
+  <!-- STEERING + WHEELS -->
+  <xacro:wheel.steering_hub side="fl" />
+  <xacro:wheel.steering_hub side="fr" />
+  <xacro:wheel.wheel side="fl" parent="fl_steering_hub_link" />
+  <xacro:wheel.wheel side="fr" parent="fr_steering_hub_link" />
+  <xacro:wheel.wheel side="rl" parent="body_link" />
+  <xacro:wheel.wheel side="rr" parent="body_link" />
+  <!-- GAZEBO PLUGINS (sim only) -->
+  <xacro:if value="$(arg use_sim)">
+    <!-- Drive and state publishing via native Gazebo plugins -->
+    <xacro:gz.ackermann_steering namespace="$(arg namespace)" />
+    <xacro:gz.joint_state_publisher namespace="$(arg namespace)" />
+    <!-- Sensors -->
+    <xacro:gz.imu reference_frame="imu_link" namespace="$(arg namespace)" />
+    <xacro:gz.rplidar reference_frame="laser" namespace="$(arg namespace)" />
+    <xacro:gz.realsense_d435 reference_frame="realsense_link" namespace="$(arg namespace)" />
+    <xacro:gz.csi_camera name="csi_front" reference_frame="csi_front_link" namespace="$(arg namespace)" />
+    <xacro:gz.csi_camera name="csi_right" reference_frame="csi_right_link" namespace="$(arg namespace)" />
+    <xacro:gz.csi_camera name="csi_back"  reference_frame="csi_back_link"  namespace="$(arg namespace)" />
+    <xacro:gz.csi_camera name="csi_left"  reference_frame="csi_left_link"  namespace="$(arg namespace)" />
+  </xacro:if>
+</robot>

File: install/qcar_description/share/qcar_description/urdf/qcar_body.urdf.xacro (robot description, xacro)
@@ -1 +1,122 @@
-/home/g16/Documents/qcarSim/src/qcar_description/urdf/qcar_body.urdf.xacro
+<?xml version="1.0" encoding="utf-8"?>
+<robot xmlns:xacro="http://www.ros.org/wiki/xacro">
+  <xacro:macro name="body" params="wheel_radius namespace">
+    <!-- ==================== BASE LINK ==================== -->
+    <link name="base_link" />
+    <joint name="base_to_body_joint" type="fixed">
+      <origin xyz="0.0 0.0 ${wheel_radius}" rpy="0.0 0.0 0.0" />
+      <parent link="base_link" />
+      <child link="body_link" />
+    </joint>
+    <!-- ==================== BODY LINK ==================== -->
+    <link name="body_link">
+      <visual>
+        <geometry>
+          <mesh filename="package://qcar_description/meshes/QCarBody.dae" scale="0.1 0.1 0.1" />
+        </geometry>
+        <material name="White">
+          <color rgba="1.0 1.0 1.0 1.0" />
+        </material>
+      </visual>
+      <collision>
+        <geometry>
+          <box size="0.38 0.12 0.10" />
+        </geometry>
+        <origin xyz="0.0 0.0 0.05" rpy="0.0 0.0 0.0" />
+      </collision>
+      <inertial>
+        <mass value="2.0" />
+        <inertia ixx="0.00387" ixy="0.0"     ixz="0.0"
+                               iyy="0.01277" iyz="0.0"
+                                             izz="0.01387" />
+        <origin xyz="0.0 0.0 0.05" rpy="0.0 0.0 0.0" />
+      </inertial>
+    </link>
+    <!-- ==================== IMU ==================== -->
+    <joint name="body_to_imu_joint" type="fixed">
+      <origin xyz="0.1278 0.0223 0.0792" rpy="0.0 0.0 0.0" />
+      <parent link="body_link" />
+      <child link="imu_link" />
+    </joint>
+    <link name="imu_link" />
+    <!-- ==================== RPLiDAR ==================== -->
+    <joint name="body_to_rplidar_joint" type="fixed">
+      <origin xyz="-0.0108 0.0 0.1696" rpy="0.0 0.0 0.0" />
+      <parent link="body_link" />
+      <child link="rplidar_link" />
+    </joint>
+    <link name="rplidar_link">
+      <visual>
+        <geometry>
+          <mesh filename="package://qcar_description/meshes/QCarLidar.dae" scale="0.1 0.1 0.1" />
+        </geometry>
+        <origin xyz="0.0 0.0 0.0" rpy="0.0 0.0 1.54" />
+        <material name="Blue">
+          <color rgba="0.2 0.2 0.8 1.0" />
+        </material>
+      </visual>
+      <collision>
+        <geometry>
+          <cylinder radius="0.035" length="0.04" />
+        </geometry>
+      </collision>
+      <inertial>
+        <mass value="0.1" />
+        <inertia ixx="0.0000418" ixy="0.0"       ixz="0.0"
+                                 iyy="0.0000418" iyz="0.0"
+                                                  izz="0.0000613" />
+      </inertial>
+    </link>
+    <!-- Laser frame (sensor reference point) -->
+    <joint name="rplidar_to_laser_joint" type="fixed">
+      <origin xyz="0.0 0.0 0.02" rpy="0.0 0.0 0.0" />
+      <parent link="rplidar_link" />
+      <child link="laser" />
+    </joint>
+    <link name="laser" />
+    <!-- ==================== REALSENSE D435 ==================== -->
+    <!-- Original d435.dae visual mesh was removed because the QCar body mesh
+         already includes the RealSense camera visually. The separate mesh
+         (models/realsense/d435.dae, no scale — already in meters) was causing
+         a duplicate camera to render on top of the body.
+         The realsense_link frame is still needed for the Gazebo depth/color
+         sensor plugins defined in qcar_gz.urdf.xacro.
+         Position from original qcar_model.xacro is xyz 0.081686 0.0 0.15445
+         relative to body_link (which sits at wheel_radius above base_link). -->
+    <joint name="body_to_realsense_joint" type="fixed">
+      <origin xyz="0.081686 0.0 0.15445" rpy="0.0 0.0 0.0" />
+      <parent link="body_link" />
+      <child link="realsense_link" />
+    </joint>
+    <link name="realsense_link" />
+    <!-- Optical frame convention Z-forward, X-right, Y-down.
+         The rpy="${-pi/2} 0 ${-pi/2}" rotates from the ROS body convention
+         (X-forward, Y-left, Z-up) into the camera optical convention.
+         If depth/color images appear flipped or rotated, check this transform. -->
+    <joint name="realsense_optical_joint" type="fixed">
+      <origin xyz="0.0 0.0 0.0" rpy="${-pi/2} 0.0 ${-pi/2}" />
+      <parent link="realsense_link" />
+      <child link="realsense_optical_frame" />
+    </joint>
+    <link name="realsense_optical_frame" />
+    <!-- ==================== CSI CAMERAS ==================== -->
+    <xacro:macro name="csi_camera_frame" params="name xyz rpy">
+      <joint name="body_to_${name}_joint" type="fixed">
+        <origin xyz="${xyz}" rpy="${rpy}" />
+        <parent link="body_link" />
+        <child link="${name}_link" />
+      </joint>
+      <link name="${name}_link" />
+      <joint name="${name}_optical_joint" type="fixed">
+        <origin xyz="0.0 0.0 0.0" rpy="${-pi/2} 0.0 ${-pi/2}" />
+        <parent link="${name}_link" />
+        <child link="${name}_optical_frame" />
+      </joint>
+      <link name="${name}_optical_frame" />
+    </xacro:macro>
+    <xacro:csi_camera_frame name="csi_front" xyz="0.19236 -0.000475 0.093029" rpy="0.0 0.0 0.0" />
+    <xacro:csi_camera_frame name="csi_right" xyz="0.12887 -0.06755 0.093029"  rpy="0.0 0.0 ${-pi/2}" />
+    <xacro:csi_camera_frame name="csi_back"  xyz="-0.16669 -0.000578 0.093029" rpy="0.0 0.0 ${pi}" />
+    <xacro:csi_camera_frame name="csi_left"  xyz="0.12784 0.052497 0.093029"  rpy="0.0 0.0 ${pi/2}" />
+  </xacro:macro>
+</robot>

File: install/qcar_description/share/qcar_description/urdf/qcar_gz.urdf.xacro (robot description, xacro)
@@ -1 +1,190 @@
-/home/g16/Documents/qcarSim/src/qcar_description/urdf/qcar_gz.urdf.xacro
+<?xml version="1.0" encoding="utf-8"?>
+<robot xmlns:xacro="http://wiki.ros.org/xacro">
+  <!-- ==================== ACKERMANN STEERING (native Gazebo plugin) ==================== -->
+  <!-- This replaces ros2_control for drive. Gazebo directly handles cmd_vel to wheel commands.
+       The plugin subscribes to a Twist message on <topic> and commands the steering/drive joints.
+       Odometry is published on <odom_topic>. -->
+  <xacro:macro name="ackermann_steering" params="namespace:=''">
+    <xacro:property name="ns" value="${namespace + '/' if namespace != '' else ''}" />
+    <gazebo>
+      <plugin filename="gz-sim-ackermann-steering-system"
+              name="gz::sim::systems::AckermannSteering">
+        <topic>${ns}cmd_vel</topic>
+        <left_steering_joint>fl_steering_joint</left_steering_joint>
+        <right_steering_joint>fr_steering_joint</right_steering_joint>
+        <left_joint>rl_wheel_joint</left_joint>
+        <right_joint>rr_wheel_joint</right_joint>
+        <kingpin_width>0.112</kingpin_width>
+        <steering_limit>0.5236</steering_limit>
+        <wheel_base>0.256</wheel_base>
+        <wheel_separation>0.112</wheel_separation>
+        <wheel_radius>0.033</wheel_radius>
+        <!-- Odom/TF disabled — OdometryPublisher plugin handles ground truth -->
+        <odom_publish_frequency>0</odom_publish_frequency>
+        <publish_odom>false</publish_odom>
+        <publish_odom_tf>false</publish_odom_tf>
+      </plugin>
+      <!-- Ground truth odometry from physics engine pose (not wheel kinematics) -->
+      <plugin filename="gz-sim-odometry-publisher-system"
+              name="gz::sim::systems::OdometryPublisher">
+        <odom_frame>odom</odom_frame>
+        <robot_base_frame>base_link</robot_base_frame>
+        <odom_topic>${ns}odom</odom_topic>
+        <tf_topic>${ns}tf</tf_topic>
+        <odom_publish_frequency>50</odom_publish_frequency>
+        <dimensions>3</dimensions>
+      </plugin>
+    </gazebo>
+  </xacro:macro>
+  <!-- ==================== JOINT STATE PUBLISHER (native Gazebo plugin) ==================== -->
+  <!-- Publishes joint states for all joints so the bridge can relay them to ROS /joint_states. -->
+  <xacro:macro name="joint_state_publisher" params="namespace:=''">
+    <xacro:property name="ns" value="${namespace + '/' if namespace != '' else ''}" />
+    <gazebo>
+      <plugin filename="gz-sim-joint-state-publisher-system"
+              name="gz::sim::systems::JointStatePublisher">
+        <topic>${ns}joint_states</topic>
+        <joint_name>fl_steering_joint</joint_name>
+        <joint_name>fr_steering_joint</joint_name>
+        <joint_name>fl_wheel_joint</joint_name>
+        <joint_name>fr_wheel_joint</joint_name>
+        <joint_name>rl_wheel_joint</joint_name>
+        <joint_name>rr_wheel_joint</joint_name>
+      </plugin>
+    </gazebo>
+  </xacro:macro>
+  <!-- ==================== GAUSS NOISE HELPER ==================== -->
+  <xacro:macro name="gauss_noise"
+    params="mean:=0.0 stddev:=0.0 bias_mean:=0.0 bias_stddev:=0.0 precision:=0.0">
+    <noise type="gaussian">
+      <mean>${mean}</mean>
+      <stddev>${stddev}</stddev>
+      <bias_mean>${bias_mean}</bias_mean>
+      <bias_stddev>${bias_stddev}</bias_stddev>
+      <precision>${precision}</precision>
+    </noise>
+  </xacro:macro>
+  <!-- ==================== IMU SENSOR ==================== -->
+  <xacro:macro name="imu" params="reference_frame namespace:=''">
+    <xacro:property name="ns" value="${namespace + '/' if namespace != '' else ''}" />
+    <gazebo reference="${reference_frame}">
+      <sensor name="${ns}imu" type="imu">
+        <always_on>true</always_on>
+        <update_rate>50</update_rate>
+        <topic>${ns}imu/data_raw</topic>
+        <visualize>false</visualize>
+        <enable_metrics>false</enable_metrics>
+        <gz_frame_id>imu_link</gz_frame_id>
+        <imu>
+          <angular_velocity>
+            <x><xacro:gauss_noise stddev="5.24e-3" bias_mean="2.0e-3" precision="1.07e-3" /></x>
+            <y><xacro:gauss_noise stddev="5.24e-3" bias_mean="2.0e-3" precision="1.07e-3" /></y>
+            <z><xacro:gauss_noise stddev="5.24e-3" bias_mean="2.0e-3" precision="1.07e-3" /></z>
+          </angular_velocity>
+          <linear_acceleration>
+            <x><xacro:gauss_noise stddev="1.86e-3" bias_mean="1.0e-3" precision="2.40e-3" /></x>
+            <y><xacro:gauss_noise stddev="1.86e-3" bias_mean="1.0e-3" precision="2.40e-3" /></y>
+            <z><xacro:gauss_noise stddev="1.86e-3" bias_mean="1.0e-3" precision="2.40e-3" /></z>
+          </linear_acceleration>
+        </imu>
+      </sensor>
+    </gazebo>
+  </xacro:macro>
+  <!-- ==================== RPLIDAR A2 ==================== -->
+  <xacro:macro name="rplidar" params="reference_frame namespace:=''">
+    <xacro:property name="ns" value="${namespace + '/' if namespace != '' else ''}" />
+    <gazebo reference="${reference_frame}">
+      <sensor name="${ns}rplidar" type="gpu_lidar">
+        <update_rate>10</update_rate>
+        <topic>${ns}scan</topic>
+        <gz_frame_id>laser</gz_frame_id>
+        <ray>
+          <scan>
+            <horizontal>
+              <samples>720</samples>
+              <resolution>1</resolution>
+              <min_angle>-${pi}</min_angle>
+              <max_angle>${pi}</max_angle>
+            </horizontal>
+          </scan>
+          <range>
+            <min>0.15</min>
+            <max>12.0</max>
+            <resolution>0.01</resolution>
+          </range>
+          <noise>
+            <type>gaussian</type>
+            <mean>0</mean>
+            <stddev>0.005</stddev>
+          </noise>
+        </ray>
+        <visualize>false</visualize>
+      </sensor>
+    </gazebo>
+  </xacro:macro>
+  <!-- ==================== REALSENSE D435 ==================== -->
+  <xacro:macro name="realsense_d435" params="reference_frame namespace:=''">
+    <xacro:property name="ns" value="${namespace + '/' if namespace != '' else ''}" />
+    <gazebo reference="${reference_frame}">
+      <!-- Color camera -->
+      <sensor name="${ns}realsense_color" type="camera">
+        <update_rate>30</update_rate>
+        <topic>${ns}realsense/color/image_raw</topic>
+        <gz_frame_id>realsense_optical_frame</gz_frame_id>
+        <camera>
+          <horizontal_fov>1.211</horizontal_fov>
+          <image>
+            <width>640</width>
+            <height>480</height>
+            <format>R8G8B8</format>
+          </image>
+          <clip>
+            <near>0.1</near>
+            <far>10.0</far>
+          </clip>
+        </camera>
+      </sensor>
+      <!-- Depth camera -->
+      <sensor name="${ns}realsense_depth" type="depth_camera">
+        <update_rate>30</update_rate>
+        <topic>${ns}realsense/depth/image_rect_raw</topic>
+        <gz_frame_id>realsense_optical_frame</gz_frame_id>
+        <camera>
+          <horizontal_fov>1.489</horizontal_fov>
+          <image>
+            <width>640</width>
+            <height>480</height>
+            <format>R_FLOAT32</format>
+          </image>
+          <clip>
+            <near>0.1</near>
+            <far>10.0</far>
+          </clip>
+        </camera>
+      </sensor>
+    </gazebo>
+  </xacro:macro>
+  <!-- ==================== CSI CAMERA ==================== -->
+  <xacro:macro name="csi_camera" params="name reference_frame namespace:=''">
+    <xacro:property name="ns" value="${namespace + '/' if namespace != '' else ''}" />
+    <gazebo reference="${reference_frame}">
+      <sensor name="${ns}${name}" type="camera">
+        <update_rate>30</update_rate>
+        <topic>${ns}${name}/image_raw</topic>
+        <gz_frame_id>${name}_optical_frame</gz_frame_id>
+        <camera>
+          <horizontal_fov>1.085</horizontal_fov>
+          <image>
+            <width>640</width>
+            <height>480</height>
+            <format>R8G8B8</format>
+          </image>
+          <clip>
+            <near>0.05</near>
+            <far>20.0</far>
+          </clip>
+        </camera>
+      </sensor>
+    </gazebo>
+  </xacro:macro>
+</robot>

File: install/qcar_description/share/qcar_description/urdf/qcar_wheels.urdf.xacro (robot description, xacro)
@@ -1 +1,131 @@
-/home/g16/Documents/qcarSim/src/qcar_description/urdf/qcar_wheels.urdf.xacro
+<?xml version="1.0" encoding="utf-8"?>
+<robot xmlns:xacro="http://www.ros.org/wiki/xacro">
+  <!-- ==================== GEOMETRY CONSTANTS ==================== -->
+  <xacro:property name="wheel_radius"    value="0.033" />
+  <xacro:property name="wheel_thickness" value="0.025" />
+  <xacro:property name="wheel_mass"      value="0.05" />
+  <!-- Wheel inertia (solid cylinder: Ixx=Iyy=m(3r^2+h^2)/12, Izz=mr^2/2) -->
+  <xacro:property name="wheel_ixx" value="0.0000162" />
+  <xacro:property name="wheel_iyy" value="0.0000162" />
+  <xacro:property name="wheel_izz" value="0.0000272" />
+  <xacro:property name="hub_mass" value="0.02" />
+  <!-- Axle positions (relative to body_link) -->
+  <xacro:property name="front_axle_x" value="0.1296" />
+  <xacro:property name="rear_axle_x"  value="-0.12765" />
+  <xacro:property name="half_track"   value="0.056" />
+  <xacro:property name="steering_limit" value="0.5236" />
+  <!-- ==================== STEERING HUB MACRO ==================== -->
+  <xacro:macro name="steering_hub" params="side">
+    <xacro:if value="${side == 'fl'}">
+      <xacro:property name="y_sign" value="1.0" />
+      <xacro:property name="hub_mesh" value="package://qcar_description/meshes/QCarSteeringHubL.dae" />
+    </xacro:if>
+    <xacro:if value="${side == 'fr'}">
+      <xacro:property name="y_sign" value="-1.0" />
+      <xacro:property name="hub_mesh" value="package://qcar_description/meshes/QCarSteeringHubR.dae" />
+    </xacro:if>
+    <joint name="${side}_steering_joint" type="revolute">
+      <parent link="body_link" />
+      <child link="${side}_steering_hub_link" />
+      <origin xyz="${front_axle_x} ${y_sign * half_track} 0.0" rpy="0.0 0.0 0.0" />
+      <axis xyz="0.0 0.0 1.0" />
+      <limit lower="${-steering_limit}" upper="${steering_limit}" effort="10.0" velocity="3.0" />
+      <dynamics damping="0.1" friction="0.0" />
+    </joint>
+    <link name="${side}_steering_hub_link">
+      <visual>
+        <geometry>
+          <mesh filename="${hub_mesh}" scale="0.1 0.1 0.1" />
+        </geometry>
+        <material name="Orange">
+          <color rgba="1.0 0.42 0.04 1.0" />
+        </material>
+      </visual>
+      <collision>
+        <geometry>
+          <sphere radius="0.01" />
+        </geometry>
+      </collision>
+      <inertial>
+        <mass value="${hub_mass}" />
+        <inertia ixx="0.0000008" ixy="0.0"       ixz="0.0"
+                                 iyy="0.0000008" iyz="0.0"
+                                                  izz="0.0000008" />
+      </inertial>
+    </link>
+  </xacro:macro>
+  <!-- ==================== WHEEL MACRO ==================== -->
+  <xacro:macro name="wheel" params="side parent">
+    <!-- Determine position and mesh orientation per side -->
+    <xacro:if value="${side == 'fl'}">
+      <xacro:property name="wheel_x" value="0.0" />
+      <xacro:property name="wheel_y" value="0.0" />
+      <xacro:property name="wheel_rpy" value="0.0 0.0 ${pi}" />
+      <xacro:property name="wheel_color" value="1.0 0.0 0.0 1.0" />
+    </xacro:if>
+    <xacro:if value="${side == 'fr'}">
+      <xacro:property name="wheel_x" value="0.0" />
+      <xacro:property name="wheel_y" value="0.0" />
+      <xacro:property name="wheel_rpy" value="0.0 0.0 0.0" />
+      <xacro:property name="wheel_color" value="1.0 0.42 0.04 1.0" />
+    </xacro:if>
+    <xacro:if value="${side == 'rl'}">
+      <xacro:property name="wheel_x" value="${rear_axle_x}" />
+      <xacro:property name="wheel_y" value="${half_track}" />
+      <xacro:property name="wheel_rpy" value="0.0 0.0 ${pi}" />
+      <xacro:property name="wheel_color" value="1.0 0.42 0.04 1.0" />
+    </xacro:if>
+    <xacro:if value="${side == 'rr'}">
+      <xacro:property name="wheel_x" value="${rear_axle_x}" />
+      <xacro:property name="wheel_y" value="${-half_track}" />
+      <xacro:property name="wheel_rpy" value="0.0 0.0 0.0" />
+      <xacro:property name="wheel_color" value="1.0 0.0 0.0 1.0" />
+    </xacro:if>
+    <joint name="${side}_wheel_joint" type="continuous">
+      <parent link="${parent}" />
+      <child link="${side}_wheel_link" />
+      <origin xyz="${wheel_x} ${wheel_y} 0.0" rpy="0.0 0.0 0.0" />
+      <axis xyz="0.0 1.0 0.0" />
+      <limit effort="1.5" velocity="30.0" />
+      <dynamics damping="0.001" friction="0.005" />
+    </joint>
+    <link name="${side}_wheel_link">
+      <visual>
+        <geometry>
+          <mesh filename="package://qcar_description/meshes/QCarWheel.dae" scale="0.1 0.1 0.1" />
+        </geometry>
+        <origin xyz="0.0 0.0 0.0" rpy="${wheel_rpy}" />
+        <material name="${side}_wheel_mat">
+          <color rgba="${wheel_color}" />
+        </material>
+      </visual>
+      <collision>
+        <geometry>
+          <cylinder radius="${wheel_radius}" length="${wheel_thickness}" />
+        </geometry>
+        <origin xyz="0.0 0.0 0.0" rpy="${pi/2} 0.0 0.0" />
+      </collision>
+      <inertial>
+        <mass value="${wheel_mass}" />
+        <inertia ixx="${wheel_ixx}" ixy="0.0"          ixz="0.0"
+                                    iyy="${wheel_iyy}" iyz="0.0"
+                                                       izz="${wheel_izz}" />
+      </inertial>
+    </link>
+    <gazebo reference="${side}_wheel_link">
+      <collision>
+        <surface>
+          <friction>
+            <ode>
+              <mu>1.0</mu>
+              <mu2>0.8</mu2>
+              <slip1>0.002</slip1>
+              <slip2>0.0</slip2>
+              <fdir1>0 0 1</fdir1>
+            </ode>
+          </friction>
+        </surface>
+      </collision>
+    </gazebo>
+  </xacro:macro>
+</robot>

File: src/qcar_description/urdf/qcar.urdf.xacro (robot description, xacro)
@@ -9,5 +9,4 @@
   <xacro:include filename="$(find qcar_description)/urdf/qcar_wheels.urdf.xacro" ns="wheel" />
   <xacro:include filename="$(find qcar_description)/urdf/qcar_gz.urdf.xacro" ns="gz" />
-  <xacro:include filename="$(find husarion_components_description)/urdf/components.urdf.xacro" ns="components" />
   <!-- PROPERTIES -->
   <xacro:property name="wheel_radius" value="0.033" />
@@ -35,9 +34,3 @@
     <xacro:gz.csi_camera name="csi_left"  reference_frame="csi_left_link"  namespace="$(arg namespace)" />
   </xacro:if>
-  <!-- EXTERNAL COMPONENTS (from husarion_components_description) -->
-  <xacro:components.create_components
-    components_config_path="$(arg components_config)"
-    namespace="$(arg namespace)"
-    use_sim="$(arg use_sim)"
-    use_tf_prefix="False" />
 </robot>
