Commit message: Sim completed for KPIs

File: src/qcar_description/urdf/qcar_gz.urdf.xacro (robot description, xacro)
@@ -20,8 +20,18 @@
         <wheel_separation>0.112</wheel_separation>
         <wheel_radius>0.033</wheel_radius>
+        <!-- Odom/TF disabled — OdometryPublisher plugin handles ground truth -->
+        <odom_publish_frequency>0</odom_publish_frequency>
+        <publish_odom>false</publish_odom>
+        <publish_odom_tf>false</publish_odom_tf>
+      </plugin>
+      <!-- Ground truth odometry from physics engine pose (not wheel kinematics) -->
+      <plugin filename="gz-sim-odometry-publisher-system"
+              name="gz::sim::systems::OdometryPublisher">
+        <odom_frame>odom</odom_frame>
+        <robot_base_frame>base_link</robot_base_frame>
         <odom_topic>${ns}odom</odom_topic>
-        <frame_id>odom</frame_id>
-        <child_frame_id>base_link</child_frame_id>
+        <tf_topic>${ns}tf</tf_topic>
         <odom_publish_frequency>50</odom_publish_frequency>
+        <dimensions>3</dimensions>
       </plugin>
     </gazebo>
